File: hardware/usb_power_meter/usb_power_meter.kicad_sch (KiCad schematic)
At the start: 35 parts, among them J1 Conn_ARM_JTAG_SWD_10, J2 USB_A, J4 USB_A, Q1 2N7002, Q2 IRML6401, U1 nRF52833-QDxx, U2 INA226, X1 32Mhz crystal, X2 32.768kHz crystal

Commit message: Add shunt resistor
Parts:
- removed R4: R_Shunt, symbol Device:R_Small
- added C18: 100 nF, Capacitor_SMD:C_0402_1005Metric, symbol Ostranna:100 nF
- added R7: 10k, Resistor_SMD:R_0201_0603Metric, symbol Ostranna:10k Resistor
- added R8: LRP12FTDSR020, Resistor_SMD:R_2512_6332Metric, symbol Ostranna:LRP12FTDSR020
Connections:
- net GND: now also C18.2
- net VBUS: now also C18.1, R8.1
- net VDD: now also R7.1
- net at Q2.2 (S), R2.1, U2.9 (Vin-): now also R8.2
- net at U1.6 (P1.09), U2.3 (~{Alert}): now also R7.2
- no-connect marks 24 -> 23
Other:
- note removed: "TODO: Replace R4 with a proper shunt resistor"
- moved on the sheet: R5, R6

Commit message: Fix INA226 power supply and use proper 4-wire connection for the shunt resistor
Connections:
- net VBUS: no longer C18.1, U2.6 (VS)
- net VDD: now also C18.1, U2.6 (VS)
Other:
- moved on the sheet: C18
Changed lines of the file:
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@@
   (junction (at 148.59 146.05) (diameter 0) (color 0 0 0 0)
   )
+  (junction (at 101.6 151.13) (diameter 0) (color 0 0 0 0)
+  )
   (junction (at 133.35 62.23) (diameter 0) (color 0 0 0 0)
   )
@@
   (junction (at 119.38 68.58) (diameter 0) (color 0 0 0 0)
   )
+  (junction (at 121.92 134.62) (diameter 0) (color 0 0 0 0)
+  )
   (junction (at 68.58 106.68) (diameter 0) (color 0 0 0 0)
   )
@@
   )
   (junction (at 86.36 97.79) (diameter 0) (color 0 0 0 0)
-  )
-  (junction (at 116.84 146.05) (diameter 0) (color 0 0 0 0)
   )
   (junction (at 186.69 120.65) (diameter 0) (color 0 0 0 0)
@@
     (stroke (width 0) (type default))
   )
-  (wire (pts (xy 116.84 146.05) (xy 116.84 151.13))
-    (stroke (width 0) (type default))
-  )
   (wire (pts (xy 180.34 120.65) (xy 186.69 120.65))
     (stroke (width 0) (type default))
   )
+  (wire (pts (xy 127 134.62) (xy 127 146.05))
+    (stroke (width 0) (type default))
+  )
   (wire (pts (xy 143.51 135.89) (xy 143.51 161.29))
     (stroke (width 0) (type default))
@@
     (stroke (width 0) (type default))
   )
-  (wire (pts (xy 127 146.05) (xy 116.84 146.05))
+  (wire (pts (xy 121.92 134.62) (xy 127 134.62))
     (stroke (width 0) (type default))
   )
@@
     (stroke (width 0) (type default))
   )
-  (wire (pts (xy 101.6 149.86) (xy 101.6 153.67))
+  (wire (pts (xy 101.6 151.13) (xy 101.6 149.86))
     (stroke (width 0) (type default))
   )
@@
     (stroke (width 0) (type default))
   )
-  (wire (pts (xy 113.03 146.05) (xy 116.84 146.05))
-    (stroke (width 0) (type default))
-  )
   (wire (pts (xy 115.57 82.55) (xy 109.22 82.55))
     (stroke (width 0) (type default))
@@
     (stroke (width 0) (type default))
   )
+  (wire (pts (xy 101.6 151.13) (xy 101.6 153.67))
+    (stroke (width 0) (type default))
+  )
   (wire (pts (xy 96.52 97.79) (xy 120.65 97.79))
     (stroke (width 0) (type default))
@@
   )
   (wire (pts (xy 116.84 163.83) (xy 107.95 163.83))
+    (stroke (width 0) (type default))
+  )
+  (wire (pts (xy 101.6 151.13) (xy 116.84 151.13))
     (stroke (width 0) (type default))
   )
@@
   (symbol (lib_id "Ostranna:4.7 uF") (at 129.54 134.62 0) (unit 1)
     (in_bom yes) (on_board yes) (dnp no)
-    (property "Reference" "C19" (at 123.19 134.62 0)
-      (effects (font (size 1.27 1.27)) (justify left))
-    )
-    (property "Value" "4.7 uF" (at 121.92 137.16 0)
+    (property "Reference" "C19" (at 129.54 137.16 0)
+      (effects (font (size 1.27 1.27)) (justify left))
+    )
+    (property "Value" "4.7 uF" (at 129.54 139.7 0)
       (effects (font (size 1.27 1.27)) (justify left))
     )
@@
     )
   )
-  (symbol (lib_id "Ostranna:100 nF") (at 113.03 149.86 0) (unit 1)
-    (in_bom yes) (on_board yes) (dnp no)
-    (property "Reference" "C18" (at 110.49 147.32 0)
-      (effects (font (size 1.27 1.27)) (justify left))
-    )
-    (property "Value" "100 nF" (at 111.76 152.4 0)
-      (effects (font (size 1.27 1.27)) (justify left))
-    )
-    (property "Footprint" "Capacitor_SMD:C_0402_1005Metric" (at 113.9952 153.67 0)
-      (effects (font (size 1.27 1.27)) hide)
-    )
-    (property "Datasheet" "~" (at 113.03 149.86 0)
-      (effects (font (size 1.27 1.27)) hide)
-    )
-    (property "LCSC" "C1525" (at 113.03 149.86 0)
-      (effects (font (size 1.27 1.27)) hide)
-    )
-    (property "LCSC type" "Basic" (at 113.03 149.86 0)
+  (symbol (lib_id "Ostranna:100 nF") (at 121.92 138.43 0) (unit 1)
+    (in_bom yes) (on_board yes) (dnp no)
+    (property "Reference" "C18" (at 119.38 135.89 0)
+      (effects (font (size 1.27 1.27)) (justify left))
+    )
+    (property "Value" "100 nF" (at 118.11 140.97 0)
+      (effects (font (size 1.27 1.27)) (justify left))
+    )
+    (property "Footprint" "Capacitor_SMD:C_0402_1005Metric" (at 122.8852 142.24 0)
+      (effects (font (size 1.27 1.27)) hide)
+    )
+    (property "Datasheet" "~" (at 121.92 138.43 0)
+      (effects (font (size 1.27 1.27)) hide)
+    )
+    (property "LCSC" "C1525" (at 121.92 138.43 0)
+      (effects (font (size 1.27 1.27)) hide)
+    )
+    (property "LCSC type" "Basic" (at 121.92 138.43 0)
       (effects (font (size 1.27 1.27)) hide)
     )
@@
         (path "/991df1c7-1ea4-4c32-892f-6236282859f6"
           (reference "C18") (unit 1)
-        )
-      )
-    )
-  )
-  (symbol (lib_id "power:VBUS") (at 116.84 146.05 0) (unit 1)
-    (in_bom yes) (on_board yes) (dnp no) (fields_autoplaced)
-    (property "Reference" "#PWR024" (at 116.84 149.86 0)
-      (effects (font (size 1.27 1.27)) hide)
-    )
-    (property "Value" "VBUS" (at 116.84 142.24 0)
-      (effects (font (size 1.27 1.27)))
-    )
-    (property "Footprint" "" (at 116.84 146.05 0)
-      (effects (font (size 1.27 1.27)) hide)
-    )
-    (property "Datasheet" "" (at 116.84 146.05 0)
-      (effects (font (size 1.27 1.27)) hide)
-    )
-    (pin "1")
-    (instances
-      (project "usb_power_meter"
-        (path "/991df1c7-1ea4-4c32-892f-6236282859f6"
-          (reference "#PWR024") (unit 1)
         )
       )
@@
   )
   (symbol (lib_id "Ostranna:INA226") (at 127 158.75 0) (unit 1)
-    (in_bom yes) (on_board yes) (dnp no) (fields_autoplaced)
-    (property "Reference" "U2" (at 128.9559 144.78 0)
-      (effects (font (size 1.27 1.27)) (justify left))
-    )
-    (property "Value" "INA226" (at 128.9559 147.32 0)
+    (in_bom yes) (on_board yes) (dnp no)
+    (property "Reference" "U2" (at 120.65 154.94 0)
+      (effects (font (size 1.27 1.27)) (justify left))
+    )
+    (property "Value" "INA226" (at 123.19 154.94 0)
       (effects (font (size 1.27 1.27)) (justify left))
     )
@@
     )
   )
-  (symbol (lib_id "power:GND") (at 113.03 153.67 0) (unit 1)
-    (in_bom yes) (on_board yes) (dnp no)
-    (property "Reference" "#PWR033" (at 113.03 160.02 0)
-      (effects (font (size 1.27 1.27)) hide)
-    )
-    (property "Value" "GND" (at 113.03 157.48 0)
-      (effects (font (size 1.27 1.27)))
-    )
-    (property "Footprint" "" (at 113.03 153.67 0)
-      (effects (font (size 1.27 1.27)) hide)
-    )
-    (property "Datasheet" "" (at 113.03 153.67 0)
+  (symbol (lib_id "power:GND") (at 121.92 142.24 0) (unit 1)
+    (in_bom yes) (on_board yes) (dnp no)
+    (property "Reference" "#PWR033" (at 121.92 148.59 0)
+      (effects (font (size 1.27 1.27)) hide)
+    )
+    (property "Value" "GND" (at 121.92 146.05 0)
+      (effects (font (size 1.27 1.27)))
+    )
+    (property "Footprint" "" (at 121.92 142.24 0)
+      (effects (font (size 1.27 1.27)) hide)
+    )
+    (property "Datasheet" "" (at 121.92 142.24 0)
       (effects (font (size 1.27 1.27)) hide)
     )
@@
         )
       )
+    )
+  )
+  (symbol (lib_id "power:VDD") (at 121.92 134.62 0) (unit 1)
+    (in_bom yes) (on_board yes) (dnp no) (fields_autoplaced)
+    (property "Reference" "#PWR024" (at 121.92 138.43 0)
+      (effects (font (size 1.27 1.27)) hide)
+    )
+    (property "Value" "VDD_nRF" (at 121.92 130.81 0)
+      (effects (font (size 1.27 1.27)))
+    )
+    (property "Footprint" "" (at 121.92 134.62 0)
+      (effects (font (size 1.27 1.27)) hide)
+    )
+    (property "Datasheet" "" (at 121.92 134.62 0)
+      (effects (font (size 1.27 1.27)) hide)
+    )
+    (pin "1")
+    (instances
+      (project "usb_power_meter"
+        (path "/991df1c7-1ea4-4c32-892f-6236282859f6"
+          (reference "#PWR024") (unit 1)
+        )
+      )

Commit message: Add an actual USB plug
Parts:
- removed J2: USB_A, Connector_USB:USB_A_Molex_67643_Horizontal, symbol Connector:USB_A
- added J2: 917-P81A202ES60201, easyeda2kicad:USB-A-SMD_917-P81A202ES60201, symbol easyeda2kicad:917-P81A202ES60201
Connections:
- net GND: now also J2.4 (GND)
- net VBUS: now also J2.1 (VCC)
- no-connect marks 23 -> 24
Changed lines of the file:
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@@
   (junction (at 96.52 88.9) (diameter 0) (color 0 0 0 0)
   )
+  (no_connect (at 25.4 166.37))
   (no_connect (at 114.3 193.04))
   (no_connect (at 173.99 92.71))
@@
   (no_connect (at 68.58 133.35))
   (no_connect (at 104.14 182.88))
+  (no_connect (at 48.26 161.29))
   (no_connect (at 162.56 130.81))
   (no_connect (at 104.14 185.42))
-  (no_connect (at 48.26 166.37))
   (no_connect (at 173.99 87.63))
   (no_connect (at 151.13 130.81))
-  (no_connect (at 38.1 173.99))
   (no_connect (at 173.99 118.11))
+  (no_connect (at 25.4 158.75))
   (no_connect (at 128.27 80.01))
   (no_connect (at 48.26 163.83))
@@
   )
   (wire (pts (xy 68.58 106.68) (xy 68.58 110.49))
+    (stroke (width 0) (type default))
+  )
+  (wire (pts (xy 48.26 166.37) (xy 48.26 171.45))
     (stroke (width 0) (type default))
   )
@@
     )
   )
-  (symbol (lib_id "power:GND") (at 40.64 173.99 0) (unit 1)
-    (in_bom yes) (on_board yes) (dnp no)
-    (property "Reference" "#PWR025" (at 40.64 180.34 0)
-      (effects (font (size 1.27 1.27)) hide)
-    )
-    (property "Value" "GND" (at 40.64 177.8 0)
-      (effects (font (size 1.27 1.27)))
-    )
-    (property "Footprint" "" (at 40.64 173.99 0)
-      (effects (font (size 1.27 1.27)) hide)
-    )
-    (property "Datasheet" "" (at 40.64 173.99 0)
-      (effects (font (size 1.27 1.27)) hide)
-    )
-    (pin "1")
-    (instances
-      (project "usb_power_meter"
-        (path "/991df1c7-1ea4-4c32-892f-6236282859f6"
-          (reference "#PWR025") (unit 1)
-        )
-      )
-    )
-  )
   (symbol (lib_id "power:VBUS") (at 67.31 158.75 0) (unit 1)
     (in_bom yes) (on_board yes) (dnp no) (fields_autoplaced)
@@
     )
   )
+  (symbol (lib_id "power:GND") (at 48.26 171.45 0) (unit 1)
+    (in_bom yes) (on_board yes) (dnp no)
+    (property "Reference" "#PWR025" (at 48.26 177.8 0)
+      (effects (font (size 1.27 1.27)) hide)
+    )
+    (property "Value" "GND" (at 48.26 175.26 0)
+      (effects (font (size 1.27 1.27)))
+    )
+    (property "Footprint" "" (at 48.26 171.45 0)
+      (effects (font (size 1.27 1.27)) hide)
+    )
+    (property "Datasheet" "" (at 48.26 171.45 0)
+      (effects (font (size 1.27 1.27)) hide)
+    )
+    (pin "1")
+    (instances
+      (project "usb_power_meter"
+        (path "/991df1c7-1ea4-4c32-892f-6236282859f6"
+          (reference "#PWR025") (unit 1)
+        )
+      )
+    )
+  )
   (symbol (lib_id "power:GND") (at 133.35 71.12 0) (unit 1)
     (in_bom yes) (on_board yes) (dnp no)
@@
     )
   )
+  (symbol (lib_id "easyeda2kicad:917-P81A202ES60201") (at 35.56 163.83 0) (mirror y) (unit 1)
+    (in_bom yes) (on_board yes) (dnp no)
+    (property "Reference" "J2" (at 36.83 154.94 0)
+      (effects (font (size 1.27 1.27)))
+    )
+    (property "Value" "917-P81A202ES60201" (at 36.83 170.18 0)
+      (effects (font (size 1.27 1.27)) hide)
+    )
+    (property "Footprint" "easyeda2kicad:USB-A-SMD_917-P81A202ES60201" (at 35.56 173.99 0)
+      (effects (font (size 1.27 1.27)) hide)
+    )
+    (property "Datasheet" "" (at 35.56 163.83 0)
+      (effects (font (size 1.27 1.27)) hide)
+    )
+    (property "Manufacturer" "精拓金" (at 35.56 176.53 0)
+      (effects (font (size 1.27 1.27)) hide)
+    )
+    (property "LCSC Part" "C2763091" (at 35.56 179.07 0)
+      (effects (font (size 1.27 1.27)) hide)
+    )
+    (pin "1")
+    (pin "2")
+    (pin "3")
+    (pin "4")
+    (pin "5")
+    (pin "6")
+    (instances
+      (project "usb_power_meter"
+        (path "/991df1c7-1ea4-4c32-892f-6236282859f6"
+          (reference "J2") (unit 1)
+        )
+      )
+    )
+  )
   (symbol (lib_id "Ostranna:1.0 pF") (at 186.69 116.84 0) (unit 1)
     (in_bom yes) (on_board yes) (dnp no)
@@
         )
       )
-    )
-  )
-  (symbol (lib_id "Connector:USB_A") (at 40.64 163.83 0) (unit 1)
-    (in_bom yes) (on_board yes) (dnp no) (fields_autoplaced)
-    (property "Reference" "J2" (at 40.64 152.4 0)
-      (effects (font (size 1.27 1.27)))
-    )
-    (property "Value" "USB_A" (at 40.64 154.94 0)
-      (effects (font (size 1.27 1.27)))
-    )
-    (property "Footprint" "Connector_USB:USB_A_Molex_67643_Horizontal" (at 44.45 165.1 0)
-      (effects (font (size 1.27 1.27)) hide)
-    )
-    (property "Datasheet" " ~" (at 44.45 165.1 0)
-      (effects (font (size 1.27 1.27)) hide)
-    )
-    (pin "1")
-    (pin "2")
-    (pin "3")
-    (pin "4")
-    (pin "5")
-    (instances
-      (project "usb_power_meter"
-        (path "/991df1c7-1ea4-4c32-892f-6236282859f6"
-          (reference "J2") (unit 1)
-        )
-      )

Commit message: Add an USB socket
Parts:
- removed J4: USB_A, Connector_USB:USB_A_Molex_67643_Horizontal, symbol Connector:USB_A
- added J4: A/F LCPTrue color1.2pillar_C42605, easyeda2kicad:USB-A-SMD_USB-M-32, symbol easyeda2kicad:A_FLCPTruecolor1.2pillar_C42605
Connections:
- net GND: now also J4.1 (GND)
- net at Q2.3 (D): now also J4.4 (VCC)
- no-connect marks 24 -> 25
Changed lines of the file:
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@@
   )
   (no_connect (at 25.4 166.37))
-  (no_connect (at 114.3 193.04))
   (no_connect (at 173.99 92.71))
   (no_connect (at 160.02 130.81))
@@
   (no_connect (at 173.99 90.17))
   (no_connect (at 173.99 97.79))
+  (no_connect (at 115.57 172.72))
   (no_connect (at 173.99 100.33))
   (no_connect (at 88.9 246.38))
@@
   (no_connect (at 173.99 120.65))
   (no_connect (at 68.58 133.35))
+  (no_connect (at 104.14 180.34))
   (no_connect (at 104.14 182.88))
   (no_connect (at 48.26 161.29))
   (no_connect (at 162.56 130.81))
-  (no_connect (at 104.14 185.42))
   (no_connect (at 173.99 87.63))
   (no_connect (at 151.13 130.81))
+  (no_connect (at 114.3 172.72))
   (no_connect (at 173.99 118.11))
   (no_connect (at 25.4 158.75))
@@
     )
   )
-  (symbol (lib_id "power:GND") (at 111.76 193.04 0) (unit 1)
-    (in_bom yes) (on_board yes) (dnp no)
-    (property "Reference" "#PWR026" (at 111.76 199.39 0)
-      (effects (font (size 1.27 1.27)) hide)
-    )
-    (property "Value" "GND" (at 111.76 196.85 0)
-      (effects (font (size 1.27 1.27)))
-    )
-    (property "Footprint" "" (at 111.76 193.04 0)
-      (effects (font (size 1.27 1.27)) hide)
-    )
-    (property "Datasheet" "" (at 111.76 193.04 0)
+  (symbol (lib_id "power:GND") (at 104.14 185.42 0) (unit 1)
+    (in_bom yes) (on_board yes) (dnp no)
+    (property "Reference" "#PWR026" (at 104.14 191.77 0)
+      (effects (font (size 1.27 1.27)) hide)
+    )
+    (property "Value" "GND" (at 104.14 189.23 0)
+      (effects (font (size 1.27 1.27)))
+    )
+    (property "Footprint" "" (at 104.14 185.42 0)
+      (effects (font (size 1.27 1.27)) hide)
+    )
+    (property "Datasheet" "" (at 104.14 185.42 0)
       (effects (font (size 1.27 1.27)) hide)
     )
@@
         (path "/991df1c7-1ea4-4c32-892f-6236282859f6"
           (reference "C6") (unit 1)
+        )
+      )
+    )
+  )
+  (symbol (lib_id "easyeda2kicad:A_FLCPTruecolor1.2pillar_C42605") (at 110.49 184.15 180) (unit 1)
+    (in_bom yes) (on_board yes) (dnp no)
+    (property "Reference" "J4" (at 113.03 181.61 0)
+      (effects (font (size 1.27 1.27)) (justify right))
+    )
+    (property "Value" "A/F LCPTrue color1.2pillar_C42605" (at 119.38 183.515 0)
+      (effects (font (size 1.27 1.27)) (justify right) hide)
+    )
+    (property "Footprint" "easyeda2kicad:USB-A-SMD_USB-M-32" (at 110.49 165.1 0)
+      (effects (font (size 1.27 1.27)) hide)
+    )
+    (property "Datasheet" "https://lcsc.com/product-detail/USB-Connectors_A-F-LCPTrue-color1-2pillar-High-temperature_C42605.html" (at 110.49 162.56 0)
+      (effects (font (size 1.27 1.27)) hide)
+    )
+    (property "Manufacturer" "精拓金" (at 110.49 160.02 0)
+      (effects (font (size 1.27 1.27)) hide)
+    )
+    (property "LCSC Part" "C42605" (at 110.49 157.48 0)
+      (effects (font (size 1.27 1.27)) hide)
+    )
+    (property "JLC Part" "Extended Part" (at 110.49 154.94 0)
+      (effects (font (size 1.27 1.27)) hide)
+    )
+    (pin "1")
+    (pin "2")
+    (pin "3")
+    (pin "4")
+    (pin "5")
+    (pin "6")
+    (instances
+      (project "usb_power_meter"
+        (path "/991df1c7-1ea4-4c32-892f-6236282859f6"
+          (reference "J4") (unit 1)
         )
       )
@@
         )
       )
-    )
-  )
-  (symbol (lib_id "Connector:USB_A") (at 111.76 182.88 0) (mirror y) (unit 1)
-    (in_bom yes) (on_board yes) (dnp no)
-    (property "Reference" "J4" (at 118.11 183.515 0)
-      (effects (font (size 1.27 1.27)) (justify right))
-    )
-    (property "Value" "USB_A" (at 118.11 180.975 0)
-      (effects (font (size 1.27 1.27)) (justify right))
-    )
-    (property "Footprint" "Connector_USB:USB_A_Molex_67643_Horizontal" (at 107.95 184.15 0)
-      (effects (font (size 1.27 1.27)) hide)
-    )
-    (property "Datasheet" " ~" (at 107.95 184.15 0)
-      (effects (font (size 1.27 1.27)) hide)
-    )
-    (pin "1")
-    (pin "2")
-    (pin "3")
-    (pin "4")
-    (pin "5")
-    (instances
-      (project "usb_power_meter"
-        (path "/991df1c7-1ea4-4c32-892f-6236282859f6"
-          (reference "J4") (unit 1)
-        )
-      )

Commit message: Add the antenna
Parts:
- added AE1: Antenna, RF_Antenna:Texas_SWRA117D_2.4GHz_Right, symbol Device:Antenna
Connections:
- net at L2.2: now also AE1.1 (A)
Other:
- note removed: "Question: Is connecting VBus and VS of INA226 okay?"
- note removed: "TODO: Add antenna"
Changed lines of the file:
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@@
     (stroke (width 0) (type default))
-  )
-  (text "TODO: Add antenna" (at 205.74 113.03 0)
-    (effects (font (size 1.27 1.27)) (justify left bottom))
-  )
-  (text "Question: Is connecting VBus and VS of INA226 okay?"
-    (at 217.17 137.16 0)
-    (effects (font (size 1.27 1.27)) (justify left bottom))
   )
   (label "EN_PWR" (at 157.48 135.89 0) (fields_autoplaced)
@@
         )
       )
+    )
+  )
+  (symbol (lib_id "Device:Antenna") (at 205.74 107.95 0) (unit 1)
+    (in_bom yes) (on_board yes) (dnp no) (fields_autoplaced)
+    (property "Reference" "AE1" (at 208.28 107.95 0)
+      (effects (font (size 1.27 1.27)) (justify left))
+    )
+    (property "Value" "Antenna" (at 208.28 110.49 0)
+      (effects (font (size 1.27 1.27)) (justify left))
+    )
+    (property "Footprint" "RF_Antenna:Texas_SWRA117D_2.4GHz_Right" (at 205.74 107.95 0)
+      (effects (font (size 1.27 1.27)) hide)
+    )
+    (property "Datasheet" "~" (at 205.74 107.95 0)
+      (effects (font (size 1.27 1.27)) hide)
+    )
+    (pin "1")
+    (instances
+      (project "usb_power_meter"
+        (path "/991df1c7-1ea4-4c32-892f-6236282859f6"
+          (reference "AE1") (unit 1)
+        )
+      )

Commit message: Add and route debugging connectors
Parts:
- removed J1: Conn_ARM_JTAG_SWD_10, Connector_PinHeader_1.27mm:PinHeader_2x05_P1.27mm_Vertical_SMD, symbol Connector:Conn_ARM_JTAG_SWD_10
- added H1: DZ254R-22-08-63, easyeda2kicad:HDR-TH_8P-P2.54-V-M-R2-C4-S2.54, symbol easyeda2kicad:DZ254R-22-08-63
- added J1: KH-1.27PH180-2X5P-L7.2-SMT, easyeda2kicad:HDR-SMD_10P-P1.27-V-M-R2-C5-LS5.5, symbol easyeda2kicad:KH-1.27PH180-2X5P-L7.2-SMT
Connections:
- net GND: now also H1.4, J1.3, J1.5, J1.9
- net VDD: now also H1.2, J1.1
- net RST: now reaches U1.16 (P0.18/~{RESET})
- net RST: now also H1.7, J1.10
- net SWDIO: now reaches U1.19 (SWDIO)
- net SWDIO: now also H1.1, J1.2
- net SWDCLK: now reaches U1.20 (SWDCLK)
- net SWDCLK: now also H1.3, J1.4
- net DBG_RX: now reaches U1.15 (P0.17)
- net DBG_RX: now also H1.5
- net DBG_TX: now reaches U1.17 (P0.20)
- net DBG_TX: now also H1.6

Commit message: Add a protection diode
Parts:
- added D1: 1N5819WS, easyeda2kicad:SOD-323_L1.8-W1.3-LS2.5-RD, symbol easyeda2kicad:1N5819WS
Connections:
- net GND: now also D1.2 (A)
- net at J4.4 (VCC), Q2.3 (D): now also D1.1 (C)
Changed lines of the file:
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@@
   (junction (at 101.6 153.67) (diameter 0) (color 0 0 0 0)
+  )
+  (junction (at 101.6 177.8) (diameter 0) (color 0 0 0 0)
   )
   (junction (at 152.4 62.23) (diameter 0) (color 0 0 0 0)
@@
     (stroke (width 0) (type default))
   )
+  (wire (pts (xy 96.52 177.8) (xy 101.6 177.8))
+    (stroke (width 0) (type default))
+  )
   (wire (pts (xy 85.09 172.72) (xy 93.98 172.72))
     (stroke (width 0) (type default))
@@
         (path "/991df1c7-1ea4-4c32-892f-6236282859f6"
           (reference "C18") (unit 1)
+        )
+      )
+    )
+  )
+  (symbol (lib_id "power:GND") (at 96.52 187.96 0) (unit 1)
+    (in_bom yes) (on_board yes) (dnp no)
+    (property "Reference" "#PWR037" (at 96.52 194.31 0)
+      (effects (font (size 1.27 1.27)) hide)
+    )
+    (property "Value" "GND" (at 96.52 191.77 0)
+      (effects (font (size 1.27 1.27)))
+    )
+    (property "Footprint" "" (at 96.52 187.96 0)
+      (effects (font (size 1.27 1.27)) hide)
+    )
+    (property "Datasheet" "" (at 96.52 187.96 0)
+      (effects (font (size 1.27 1.27)) hide)
+    )
+    (pin "1")
+    (instances
+      (project "usb_power_meter"
+        (path "/991df1c7-1ea4-4c32-892f-6236282859f6"
+          (reference "#PWR037") (unit 1)
         )
       )
@@
         )
       )
+    )
+  )
+  (symbol (lib_id "easyeda2kicad:1N5819WS") (at 96.52 182.88 270) (unit 1)
+    (in_bom yes) (on_board yes) (dnp no)
+    (property "Reference" "D1" (at 91.44 182.88 90)
+      (effects (font (size 1.27 1.27)) (justify left))
+    )
+    (property "Value" "1N5819WS" (at 100.33 184.405 90)
+      (effects (font (size 1.27 1.27)) (justify left) hide)
+    )
+    (property "Footprint" "easyeda2kicad:SOD-323_L1.8-W1.3-LS2.5-RD" (at 88.9 182.88 0)
+      (effects (font (size 1.27 1.27)) hide)
+    )
+    (property "Datasheet" "https://lcsc.com/product-detail/Others_B5819WS_C191023.html" (at 86.36 182.88 0)
+      (effects (font (size 1.27 1.27)) hide)
+    )
+    (property "Manufacturer" "Hottech(合科泰)" (at 83.82 182.88 0)
+      (effects (font (size 1.27 1.27)) hide)
+    )
+    (property "LCSC Part" "C191023" (at 81.28 182.88 0)
+      (effects (font (size 1.27 1.27)) hide)
+    )
+    (property "JLC Part" "Basic Part" (at 78.74 182.88 0)
+      (effects (font (size 1.27 1.27)) hide)
+    )
+    (pin "1")
+    (pin "2")
+    (instances
+      (project "usb_power_meter"
+        (path "/991df1c7-1ea4-4c32-892f-6236282859f6"
+          (reference "D1") (unit 1)
+        )
+      )
