File: hardware/usb_power_meter/usb_power_meter.kicad_sch (KiCad schematic)
At the start: 40 parts, among them J1 KH-1.27PH180-2X5P-L7.2-SMT, J2 917-P81A202ES60201, J4 A/F LCPTrue color1.2pillar_C4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, Q1 2N7002, Q2 IRML6401, U1 nRF52833-QDxx, U2 INA226, X1 32Mhz crystal, X2 32.768kHz crystal

Commit message: Add switch and LED
Parts:
- added LED1: 0805G (Green), easyeda2kicad:LED0805-R-RD, symbol easyeda2kicad:0805G(Green)
- added R4: 100R Resistor, Resistor_SMD:R_0603_1608Metric, symbol Ostranna:100R Resistor
- added SW1: TS-1187A-B-A-B, easyeda2kicad:SW-SMD_4P-L5.1-W5.1-P3.70-LS6.5-TL-2, symbol easyeda2kicad:TS-1187A-B-A-B
Connections:
- net GND: now also SW1.3 (C)
- net VDD: now also R4.2
- net at U1.35 (AIN6/P0.30): now also SW1.1 (A)
- net at U1.36 (AIN7/P0.31): now also LED1.2 (K)
- new net: LED1.1 (A), R4.1
Changed lines of the file:
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@@
   (no_connect (at 40.64 45.72))
   (no_connect (at 134.62 130.81))
-  (no_connect (at 173.99 90.17))
   (no_connect (at 39.37 73.66))
   (no_connect (at 173.99 97.79))
@@
   (no_connect (at 132.08 130.81))
   (no_connect (at 173.99 120.65))
+  (no_connect (at 193.04 102.87))
   (no_connect (at 104.14 180.34))
+  (no_connect (at 193.04 95.25))
   (no_connect (at 104.14 182.88))
   (no_connect (at 48.26 161.29))
   (no_connect (at 40.64 48.26))
-  (no_connect (at 173.99 87.63))
   (no_connect (at 151.13 130.81))
   (no_connect (at 114.3 172.72))
@@
     (stroke (width 0) (type default))
   )
+  (wire (pts (xy 196.85 87.63) (xy 203.2 87.63))
+    (stroke (width 0) (type default))
+  )
   (wire (pts (xy 162.56 130.81) (xy 162.56 135.89))
     (stroke (width 0) (type default))
@@
     (stroke (width 0) (type default))
   )
+  (wire (pts (xy 173.99 90.17) (xy 179.07 90.17))
+    (stroke (width 0) (type default))
+  )
+  (wire (pts (xy 179.07 87.63) (xy 173.99 87.63))
+    (stroke (width 0) (type default))
+  )
   (wire (pts (xy 143.51 130.81) (xy 143.51 135.89))
     (stroke (width 0) (type default))
@@
     (stroke (width 0) (type default))
   )
+  (wire (pts (xy 179.07 95.25) (xy 182.88 95.25))
+    (stroke (width 0) (type default))
+  )
   (wire (pts (xy 120.65 90.17) (xy 115.57 90.17))
     (stroke (width 0) (type default))
@@
   )
   (wire (pts (xy 137.16 158.75) (xy 146.05 158.75))
+    (stroke (width 0) (type default))
+  )
+  (wire (pts (xy 179.07 90.17) (xy 179.07 95.25))
     (stroke (width 0) (type default))
   )
@@
   (label "DBG_RX" (at 29.21 71.12 180) (fields_autoplaced)
     (effects (font (size 1.27 1.27)) (justify right bottom))
+  )
+  (symbol (lib_id "easyeda2kicad:0805G(Green)") (at 184.15 87.63 0) (unit 1)
+    (in_bom yes) (on_board yes) (dnp no) (fields_autoplaced)
+    (property "Reference" "LED1" (at 182.755 80.01 0)
+      (effects (font (size 1.27 1.27)))
+    )
+    (property "Value" "0805G (Green)" (at 182.755 82.55 0)
+      (effects (font (size 1.27 1.27)))
+    )
+    (property "Footprint" "easyeda2kicad:LED0805-R-RD" (at 184.15 95.25 0)
+      (effects (font (size 1.27 1.27)) hide)
+    )
+    (property "Datasheet" "https://lcsc.com/product-detail/Light-Emitting-Diodes-LED_Green-0805-Highlighted_C2297.html" (at 184.15 97.79 0)
+      (effects (font (size 1.27 1.27)) hide)
+    )
+    (property "Manufacturer" "KENTO" (at 184.15 100.33 0)
+      (effects (font (size 1.27 1.27)) hide)
+    )
+    (property "LCSC Part" "C2297" (at 184.15 102.87 0)
+      (effects (font (size 1.27 1.27)) hide)
+    )
+    (property "JLC Part" "Basic Part" (at 184.15 105.41 0)
+      (effects (font (size 1.27 1.27)) hide)
+    )
+    (pin "1")
+    (pin "2")
+    (instances
+      (project "usb_power_meter"
+        (path "/991df1c7-1ea4-4c32-892f-6236282859f6"
+          (reference "LED1") (unit 1)
+        )
+      )
+    )
   )
   (symbol (lib_id "Ostranna:12 pF") (at 73.66 102.87 90) (unit 1)
@@
         (path "/991df1c7-1ea4-4c32-892f-6236282859f6"
           (reference "#PWR015") (unit 1)
+        )
+      )
+    )
+  )
+  (symbol (lib_id "power:VDD") (at 203.2 87.63 0) (unit 1)
+    (in_bom yes) (on_board yes) (dnp no) (fields_autoplaced)
+    (property "Reference" "#PWR038" (at 203.2 91.44 0)
+      (effects (font (size 1.27 1.27)) hide)
+    )
+    (property "Value" "VDD_nRF" (at 203.2 83.82 0)
+      (effects (font (size 1.27 1.27)))
+    )
+    (property "Footprint" "" (at 203.2 87.63 0)
+      (effects (font (size 1.27 1.27)) hide)
+    )
+    (property "Datasheet" "" (at 203.2 87.63 0)
+      (effects (font (size 1.27 1.27)) hide)
+    )
+    (pin "1")
+    (instances
+      (project "usb_power_meter"
+        (path "/991df1c7-1ea4-4c32-892f-6236282859f6"
+          (reference "#PWR038") (unit 1)
         )
       )
@@
     )
   )
+  (symbol (lib_id "power:GND") (at 182.88 102.87 0) (unit 1)
+    (in_bom yes) (on_board yes) (dnp no)
+    (property "Reference" "#PWR039" (at 182.88 109.22 0)
+      (effects (font (size 1.27 1.27)) hide)
+    )
+    (property "Value" "GND" (at 182.88 106.68 0)
+      (effects (font (size 1.27 1.27)))
+    )
+    (property "Footprint" "" (at 182.88 102.87 0)
+      (effects (font (size 1.27 1.27)) hide)
+    )
+    (property "Datasheet" "" (at 182.88 102.87 0)
+      (effects (font (size 1.27 1.27)) hide)
+    )
+    (pin "1")
+    (instances
+      (project "usb_power_meter"
+        (path "/991df1c7-1ea4-4c32-892f-6236282859f6"
+          (reference "#PWR039") (unit 1)
+        )
+      )
+    )
+  )
   (symbol (lib_id "power:VDD") (at 152.4 62.23 0) (unit 1)
     (in_bom yes) (on_board yes) (dnp no)
@@
         (path "/991df1c7-1ea4-4c32-892f-6236282859f6"
           (reference "C1") (unit 1)
+        )
+      )
+    )
+  )
+  (symbol (lib_id "Ostranna:100R Resistor") (at 193.04 87.63 90) (unit 1)
+    (in_bom yes) (on_board yes) (dnp no) (fields_autoplaced)
+    (property "Reference" "R4" (at 193.04 82.55 90)
+      (effects (font (size 1.27 1.27)))
+    )
+    (property "Value" "100R Resistor" (at 193.04 85.09 90)
+      (effects (font (size 1.27 1.27)))
+    )
+    (property "Footprint" "Resistor_SMD:R_0603_1608Metric" (at 193.04 89.408 90)
+      (effects (font (size 1.27 1.27)) hide)
+    )
+    (property "Datasheet" "~" (at 193.04 87.63 0)
+      (effects (font (size 1.27 1.27)) hide)
+    )
+    (property "LCSC" "C22775" (at 193.04 87.63 0)
+      (effects (font (size 1.27 1.27)) hide)
+    )
+    (pin "1")
+    (pin "2")
+    (instances
+      (project "usb_power_meter"
+        (path "/991df1c7-1ea4-4c32-892f-6236282859f6"
+          (reference "R4") (unit 1)
         )
       )
@@
         )
       )
+    )
+  )
+  (symbol (lib_id "easyeda2kicad:TS-1187A-B-A-B") (at 187.96 97.79 0) (unit 1)
+    (in_bom yes) (on_board yes) (dnp no)
+    (property "Reference" "SW1" (at 191.77 99.06 0)
+      (effects (font (size 1.27 1.27)))
+    )
+    (property "Value" "TS-1187A-B-A-B" (at 187.96 93.98 0)
+      (effects (font (size 1.27 1.27)) hide)
+    )
+    (property "Footprint" "easyeda2kicad:SW-SMD_4P-L5.1-W5.1-P3.70-LS6.5-TL-2" (at 187.96 110.49 0)
+      (effects (font (size 1.27 1.27)) hide)
+    )
+    (property "Datasheet" "https://lcsc.com/product-detail/Tactile-Switches_XKB-Enterprise-TS-1187-B-A-A_C318884.html" (at 187.96 113.03 0)
+      (effects (font (size 1.27 1.27)) hide)
+    )
+    (property "Manufacturer" "XKB Connectivity(中国星坤)" (at 187.96 115.57 0)
+      (effects (font (size 1.27 1.27)) hide)
+    )
+    (property "LCSC Part" "C318884" (at 187.96 118.11 0)
+      (effects (font (size 1.27 1.27)) hide)
+    )
+    (property "JLC Part" "Basic Part" (at 187.96 120.65 0)
+      (effects (font (size 1.27 1.27)) hide)
+    )
+    (pin "1")
+    (pin "2")
+    (pin "3")
+    (pin "4")
+    (instances
+      (project "usb_power_meter"
+        (path "/991df1c7-1ea4-4c32-892f-6236282859f6"
+          (reference "SW1") (unit 1)
+        )
+      )
